File: Ecocar_onboarding/Onboarding - Copy/Ecocar on boarding.kicad_sch (KiCad schematic)
At the start: 50 parts, among them J1 Conn_01x04_Socket, J2 USB_C_Receptacle_USB2.0_16P, J3 Conn_01x04_Socket, J4 Conn_01x04_MountingPin, J5 Conn_01x04_MountingPin, J6 Conn_01x04_MountingPin, SW1 SW_SPDT, U1 AMS1117-3.3, U2 STM32F103C8T6, U3 BME280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

Commit message: Revision 2 upload
Parts:
- added D? (x5): LED_B, LED_SMD:LED_0603_1608Metric_Pad1.05x0.95mm_HandSolder, symbol Device:LED
- added R? (x5): 1k5, Resistor_SMD:R_0805_2012Metric_Pad1.20x1.40mm_HandSolder, symbol Device:R
Connections:
- net GND: now also D?.1 (K), D?.1 (K), D?.1 (K), D?.1 (K), D?.1 (K)
- net at U2.27 (PB14): now also R?.1
- net at U2.28 (PB15): now also R?.1
- net at U2.29 (PA8): now also R?.1
- net at U2.30 (PA9): now also R?.1
- net at U2.31 (PA10): now also R?.1
- new net: D?.2 (A), R?.2 (x5)
- no-connect marks 39 -> 34
Other:
- moved on the sheet: R5
